File: 12V_3A_supply.sch (KiCad schematic (older format))
At the start: 15 parts

Commit message: done sch and all fotprints
Parts:
- removed D?: D, symbol D
- removed R?: 976, Resistors_SMD:R_0402, symbol R
- added D1: STPS20M100S, TO_SOT_Packages_SMD:TO-263-2, symbol D_Schottky_AKA
- L1: renamed from L?; value L -> 16uH; footprint (none) -> Inductors_SMD:L_Wuerth_HCI-1050
- gave numbers to parts that had none: 12
Connections:
- net labels added: +12P
- net labels removed: +12V
- wire segments 38 -> 41
- no-connect marks 0 -> 2
Changed lines of the file:
@@
 LIBS:valves
 LIBS:MB_DEVICE
+LIBS:power_board-cache
 EELAYER 25 0
 EELAYER END
@@
 $EndDescr
 $Comp
-L TPS54561 U?
+L TPS54561 U1
 U 1 1 5AA6E6E6
 P 5450 3400
-F 0 "U?" H 5250 3900 60  0000 C CNN
+F 0 "U1" H 5250 3900 60  0000 C CNN
 F 1 "TPS54561" H 5400 3050 60  0000 C CNN
 F 2 "MB_LIB:TPS54561" H 5450 3400 60  0001 C CNN
@@
 Connection ~ 4900 3650
 $Comp
-L GND #PWR?
+L GND #PWR023
 U 1 1 5AA6E74F
 P 4900 4350
-F 0 "#PWR?" H 4900 4100 50  0001 C CNN
+F 0 "#PWR023" H 4900 4100 50  0001 C CNN
 F 1 "GND" H 4900 4200 50  0000 C CNN
 F 2 "" H 4900 4350 50  0001 C CNN
@@
 $EndComp
 $Comp
-L C C?
+L C C11
 U 1 1 5AA6E768
 P 3450 2600
-F 0 "C?" H 3475 2700 50  0000 L CNN
+F 0 "C11" H 3475 2700 50  0000 L CNN
 F 1 "3.3uF100V" H 3475 2500 50  0000 L CNN
 F 2 "Capacitors_SMD:C_1206" H 3488 2450 50  0001 C CNN
@@
 $EndComp
 $Comp
-L C C?
+L C C12
 U 1 1 5AA6E7A3
 P 3900 3900
-F 0 "C?" H 3925 4000 50  0000 L CNN
+F 0 "C12" H 3925 4000 50  0000 L CNN
 F 1 "750pF50V" V 3850 3450 50  0000 L CNN
 F 2 "Capacitors_SMD:C_0402" H 3938 3750 50  0001 C CNN
@@
 $EndComp
 $Comp
-L C C?
+L C C13
 U 1 1 5AA6E7C6
 P 4150 3650
-F 0 "C?" H 4175 3750 50  0000 L CNN
+F 0 "C13" H 4175 3750 50  0000 L CNN
 F 1 "6.8pF100V" V 4100 3200 50  0000 L CNN
 F 2 "Capacitors_SMD:C_0603" H 4188 3500 50  0001 C CNN
@@
 $EndComp
 $Comp
-L C C?
+L C C14
 U 1 1 5AA6E7E8
 P 4450 3700
-F 0 "C?" H 4475 3800 50  0000 L CNN
+F 0 "C14" H 4475 3800 50  0000 L CNN
 F 1 "2.7nF50V" V 4400 3300 50  0000 L CNN
 F 2 "Capacitors_SMD:C_0805" H 4488 3550 50  0001 C CNN
@@
 $EndComp
 $Comp
-L R R?
+L R R1
 U 1 1 5AA6E80A
 P 3900 3450
-F 0 "R?" V 3980 3450 50  0000 C CNN
+F 0 "R1" V 3980 3450 50  0000 C CNN
 F 1 "61.9K" V 3900 3450 50  0000 C CNN
 F 2 "Resistors_SMD:R_0402" V 3830 3450 50  0001 C CNN
@@
 $EndComp
 $Comp
-L R R?
+L R R2
 U 1 1 5AA6E84B
 P 4700 3700
-F 0 "R?" V 4780 3700 50  0000 C CNN
+F 0 "R2" V 4780 3700 50  0000 C CNN
 F 1 "143k" V 4700 3700 50  0000 C CNN
 F 2 "Resistors_SMD:R_0402" V 4630 3700 50  0001 C CNN
@@
 $EndComp
 $Comp
-L C C?
+L C C15
 U 1 1 5AA6E89F
 P 6300 3150
-F 0 "C?" H 6325 3250 50  0000 L CNN
+F 0 "C15" H 6325 3250 50  0000 L CNN
 F 1 "100nF" V 6250 2850 50  0000 L CNN
 F 2 "Capacitors_SMD:C_0402" H 6338 3000 50  0001 C CNN
@@
 $EndComp
 $Comp
-L R R?
+L R R3
 U 1 1 5AA6E921
 P 7000 3350
-F 0 "R?" V 7080 3350 50  0000 C CNN
+F 0 "R3" V 7080 3350 50  0000 C CNN
 F 1 "147k" V 7000 3350 50  0000 C CNN
 F 2 "Resistors_SMD:R_0402" V 6930 3350 50  0001 C CNN
@@
 $EndComp
 $Comp
-L R R?
+L R R4
 U 1 1 5AA6E9CE
 P 7000 3750
-F 0 "R?" V 7080 3750 50  0000 C CNN
+F 0 "R4" V 7080 3750 50  0000 C CNN
 F 1 "10.5k" V 7000 3750 50  0000 C CNN
 F 2 "Resistors_SMD:R_0402" V 6930 3750 50  0001 C CNN
@@
 $EndComp
 $Comp
-L +48V #PWR?
+L +48V #PWR024
 U 1 1 5AA6EAEE
 P 3450 2350
-F 0 "#PWR?" H 3450 2200 50  0001 C CNN
+F 0 "#PWR024" H 3450 2200 50  0001 C CNN
 F 1 "+48V" H 3450 2490 50  0000 C CNN
 F 2 "" H 3450 2350 50  0001 C CNN
@@
 $EndComp
 $Comp
-L +48V #PWR?
+L +48V #PWR025
 U 1 1 5AA6EB2F
 P 4900 2950
-F 0 "#PWR?" H 4900 2800 50  0001 C CNN
+F 0 "#PWR025" H 4900 2800 50  0001 C CNN
 F 1 "+48V" H 4900 3090 50  0000 C CNN
 F 2 "" H 4900 2950 50  0001 C CNN
@@
 $EndComp
 $Comp
-L GND #PWR?
+L GND #PWR026
 U 1 1 5AA6EB62
 P 3450 2850
-F 0 "#PWR?" H 3450 2600 50  0001 C CNN
+F 0 "#PWR026" H 3450 2600 50  0001 C CNN
 F 1 "GND" H 3450 2700 50  0000 C CNN
 F 2 "" H 3450 2850 50  0001 C CNN
@@
 	4700 3850 4700 4350
 $Comp
-L GND #PWR?
+L GND #PWR027
 U 1 1 5AA6EECF
 P 4700 4350
-F 0 "#PWR?" H 4700 4100 50  0001 C CNN
+F 0 "#PWR027" H 4700 4100 50  0001 C CNN
 F 1 "GND" H 4700 4200 50  0000 C CNN
 F 2 "" H 4700 4350 50  0001 C CNN
@@
 $EndComp
 $Comp
-L GND #PWR?
+L GND #PWR028
 U 1 1 5AA6EEF8
 P 4450 4350
-F 0 "#PWR?" H 4450 4100 50  0001 C CNN
+F 0 "#PWR028" H 4450 4100 50  0001 C CNN
 F 1 "GND" H 4450 4200 50  0000 C CNN
 F 2 "" H 4450 4350 50  0001 C CNN
@@
 $EndComp
 $Comp
-L GND #PWR?
+L GND #PWR029
 U 1 1 5AA6EF21
 P 4150 4350
-F 0 "#PWR?" H 4150 4100 50  0001 C CNN
+F 0 "#PWR029" H 4150 4100 50  0001 C CNN
 F 1 "GND" H 4150 4200 50  0000 C CNN
 F 2 "" H 4150 4350 50  0001 C CNN
@@
 $EndComp
 $Comp
-L GND #PWR?
+L GND #PWR030
 U 1 1 5AA6EF4A
 P 3900 4350
-F 0 "#PWR?" H 3900 4100 50  0001 C CNN
+F 0 "#PWR030" H 3900 4100 50  0001 C CNN
 F 1 "GND" H 3900 4200 50  0000 C CNN
 F 2 "" H 3900 4350 50  0001 C CNN
@@
 	1    0    0    -1
 $EndComp
-$Comp
-L R R?
-U 1 1 5AA6F18F
-P 6100 2850
-F 0 "R?" V 6180 2850 50  0000 C CNN
-F 1 "976" V 6100 2850 50  0000 C CNN
-F 2 "Resistors_SMD:R_0402" V 6030 2850 50  0001 C CNN
-F 3 "" H 6100 2850 50  0001 C CNN
-	1    6100 2850
-	1    0    0    -1
-$EndComp
-Wire Wire Line
-	6000 3050 6100 3050
-Wire Wire Line
-	6100 3050 6100 3000
-Wire Wire Line
-	6100 2700 6450 2700
 Wire Wire Line
 	6000 3150 6150 3150
@@
 	6450 3150 6600 3150
 $Comp
-L L L?
+L L L1
 U 1 1 5AA6F2C2
 P 6750 3150
-F 0 "L?" V 6700 3150 50  0000 C CNN
-F 1 "L" V 6825 3150 50  0000 C CNN
-F 2 "" H 6750 3150 50  0001 C CNN
-F 3 "" H 6750 3150 50  0001 C CNN
+F 0 "L1" V 6700 3150 50  0000 C CNN
+F 1 "16uH" V 6825 3150 50  0000 C CNN
+F 2 "Inductors_SMD:L_Wuerth_HCI-1050" H 6750 3150 50  0001 C CNN
+F 3 "http://katalog.we-online.de/pbs/datasheet/7443251600.pdf" H 6750 3150 50  0001 C CNN
 	1    6750 3150
 	0    -1   -1   0
@@
 	7000 3150 7000 3200
 Wire Wire Line
-	6000 3550 7000 3550
-Wire Wire Line
 	7000 3500 7000 3600
 Connection ~ 7000 3550
 $Comp
-L CP C?
+L CP C16
 U 1 1 5AA6F477
 P 7250 3500
-F 0 "C?" H 7275 3600 50  0000 L CNN
+F 0 "C16" H 7275 3600 50  0000 L CNN
 F 1 "4.7uF" H 7275 3400 50  0000 L CNN
 F 2 "" H 7288 3350 50  0001 C CNN
@@
 	7250 3650 7250 4350
 $Comp
-L R R?
+L R R5
 U 1 1 5AA6F613
 P 7550 3500
-F 0 "R?" V 7630 3500 50  0000 C CNN
+F 0 "R5" V 7630 3500 50  0000 C CNN
 F 1 "4" V 7550 3500 50  0000 C CNN
 F 2 "Resistors_SMD:R_0402" V 7480 3500 50  0001 C CNN
@@
 	6500 3250 6500 3150
 Connection ~ 6500 3150
-$Comp
-L D D?
-U 1 1 5AA6F774
-P 6550 3350
-F 0 "D?" H 6550 3450 50  0000 C CNN
-F 1 "D" H 6550 3250 50  0000 C CNN
-F 2 "" H 6550 3350 50  0001 C CNN
-F 3 "" H 6550 3350 50  0001 C CNN
-	1    6550 3350
-	0    1    1    0
-$EndComp
 Wire Wire Line
 	6550 3150 6550 3200
 Connection ~ 6550 3150
-Wire Wire Line
-	6550 3500 6550 4350
-$Comp
-L GND #PWR?
+$Comp
+L GND #PWR031
 U 1 1 5AA6F863
 P 6550 4350
-F 0 "#PWR?" H 6550 4100 50  0001 C CNN
+F 0 "#PWR031" H 6550 4100 50  0001 C CNN
 F 1 "GND" H 6550 4200 50  0000 C CNN
 F 2 "" H 6550 4350 50  0001 C CNN
@@
 	7000 3900 7000 4350
 $Comp
-L GND #PWR?
+L GND #PWR032
 U 1 1 5AA6F9CD
 P 7000 4350
-F 0 "#PWR?" H 7000 4100 50  0001 C CNN
+F 0 "#PWR032" H 7000 4100 50  0001 C CNN
 F 1 "GND" H 7000 4200 50  0000 C CNN
 F 2 "" H 7000 4350 50  0001 C CNN
@@
 $EndComp
 $Comp
-L GND #PWR?
+L GND #PWR033
 U 1 1 5AA6FA05
 P 7250 4350
-F 0 "#PWR?" H 7250 4100 50  0001 C CNN
+F 0 "#PWR033" H 7250 4100 50  0001 C CNN
 F 1 "GND" H 7250 4200 50  0000 C CNN
 F 2 "" H 7250 4350 50  0001 C CNN
@@
 $EndComp
 $Comp
-L GND #PWR?
+L GND #PWR034
 U 1 1 5AA6FA3D
 P 7550 4350
-F 0 "#PWR?" H 7550 4100 50  0001 C CNN
+F 0 "#PWR034" H 7550 4100 50  0001 C CNN
 F 1 "GND" H 7550 4200 50  0000 C CNN
 F 2 "" H 7550 4350 50  0001 C CNN
@@
 Connection ~ 7550 3150
 $Comp
-L +12V #PWR?
-U 1 1 5AA6FDF2
+L D_Schottky_AKA D1
+U 1 1 5AA80853
+P 6550 3350
+F 0 "D1" H 6550 3450 50  0000 C CNN
+F 1 "STPS20M100S" H 6750 3250 50  0000 C CNN
+F 2 "TO_SOT_Packages_SMD:TO-263-2" H 6550 3350 50  0001 C CNN
+F 3 "http://www.st.com/content/ccc/resource/technical/document/datasheet/group2/8f/d3/41/ea/82/b2/4b/5a/CD00228904/files/CD00228904.pdf/jcr:content/translations/en.CD00228904.pdf" H 6550 3350 50  0001 C CNN
+	1    6550 3350
+	0    1    1    0
+$EndComp
+Wire Wire Line
+	6550 3550 6550 4350
+Wire Wire Line
+	6650 3550 6650 4250
+Wire Wire Line
+	6650 4250 6550 4250
+Connection ~ 6550 4250
+Wire Wire Line
+	7000 3550 6800 3550
+Wire Wire Line
+	6800 3550 6800 3950
+Wire Wire Line
+	6800 3950 6150 3950
+Wire Wire Line
+	6150 3950 6150 3550
+Wire Wire Line
+	6150 3550 6000 3550
+NoConn ~ 4950 3150
+NoConn ~ 6000 3050
+$Comp
+L +12P #PWR035
+U 1 1 5AA81E40
 P 7750 3100
-F 0 "#PWR?" H 7750 2950 50  0001 C CNN
-F 1 "+12V" H 7750 3240 50  0000 C CNN
+F 0 "#PWR035" H 7750 2950 50  0001 C CNN
+F 1 "+12P" H 7750 3240 50  0000 C CNN
 F 2 "" H 7750 3100 50  0001 C CNN
 F 3 "" H 7750 3100 50  0001 C CNN
