File: power_board.sch (KiCad schematic (older format))
At the start: 26 parts

Commit message: done sch and all fotprints
Parts:
- C1: renamed from C?; footprint (none) -> Capacitor_THT:CP_Radial_D10.0mm_P5.00mm; MPN (none) -> 565-4315-ND
- C10, C8: renamed from C?; footprint Capacitors_THT:CP_Radial_D35.0mm_P10.00mm_SnapIn -> Capacitor_THT:CP_Radial_D10.0mm_P5.00mm
- C2, C3, C5, C6, C7, C9: renamed from C?; footprint (none) -> Capacitor_THT:CP_Radial_D10.0mm_P5.00mm
- J1, J10, J11, J12, J13, J14, J15, J16, J2, J3, J4, J5, J6, J7, J8, J9: renamed from J?; footprint (none) -> MB_LIB:via
- gave numbers to parts that had none: 1
