File: power_board.sch (KiCad schematic (older format))
At the start: 32 parts, among them J1 Conn_01x01, J10 Conn_01x01, J11 Conn_01x01, J12 Conn_01x01, J13 Conn_01x01, J14 Conn_01x01, J15 Conn_01x01, J16 Conn_01x01, J2 Conn_01x01, J3 Conn_01x01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

Commit message: first pcb layout
Parts:
- J1, J11, J13, J15, J3, J5, J7, J9: footprint MB_LIB:via -> MB_LIB:via_sq
- gave numbers to parts that had none: 6
Changed lines of the file:
@@
 F 0 "J1" H 6350 2050 50  0000 C CNN
 F 1 "Conn_01x01" H 6350 1850 50  0000 C CNN
-F 2 "MB_LIB:via" H 6350 1950 50  0001 C CNN
+F 2 "MB_LIB:via_sq" H 6350 1950 50  0001 C CNN
 F 3 "" H 6350 1950 50  0001 C CNN
 	1    6350 1950
@@
 F 0 "J3" H 6650 2050 50  0000 C CNN
 F 1 "Conn_01x01" H 6650 1850 50  0000 C CNN
-F 2 "MB_LIB:via" H 6650 1950 50  0001 C CNN
+F 2 "MB_LIB:via_sq" H 6650 1950 50  0001 C CNN
 F 3 "" H 6650 1950 50  0001 C CNN
 	1    6650 1950
@@
 F 0 "J5" H 6950 2050 50  0000 C CNN
 F 1 "Conn_01x01" H 6950 1850 50  0000 C CNN
-F 2 "MB_LIB:via" H 6950 1950 50  0001 C CNN
+F 2 "MB_LIB:via_sq" H 6950 1950 50  0001 C CNN
 F 3 "" H 6950 1950 50  0001 C CNN
 	1    6950 1950
@@
 F 0 "J7" H 7250 2050 50  0000 C CNN
 F 1 "Conn_01x01" H 7250 1850 50  0000 C CNN
-F 2 "MB_LIB:via" H 7250 1950 50  0001 C CNN
+F 2 "MB_LIB:via_sq" H 7250 1950 50  0001 C CNN
 F 3 "" H 7250 1950 50  0001 C CNN
 	1    7250 1950
@@
 F 0 "J9" H 7550 2050 50  0000 C CNN
 F 1 "Conn_01x01" H 7550 1850 50  0000 C CNN
-F 2 "MB_LIB:via" H 7550 1950 50  0001 C CNN
+F 2 "MB_LIB:via_sq" H 7550 1950 50  0001 C CNN
 F 3 "" H 7550 1950 50  0001 C CNN
 	1    7550 1950
@@
 F 0 "J11" H 7850 2050 50  0000 C CNN
 F 1 "Conn_01x01" H 7850 1850 50  0000 C CNN
-F 2 "MB_LIB:via" H 7850 1950 50  0001 C CNN
+F 2 "MB_LIB:via_sq" H 7850 1950 50  0001 C CNN
 F 3 "" H 7850 1950 50  0001 C CNN
 	1    7850 1950
@@
 F 0 "J13" H 8150 2050 50  0000 C CNN
 F 1 "Conn_01x01" H 8150 1850 50  0000 C CNN
-F 2 "MB_LIB:via" H 8150 1950 50  0001 C CNN
+F 2 "MB_LIB:via_sq" H 8150 1950 50  0001 C CNN
 F 3 "" H 8150 1950 50  0001 C CNN
 	1    8150 1950
@@
 F 0 "J15" H 8450 2050 50  0000 C CNN
 F 1 "Conn_01x01" H 8450 1850 50  0000 C CNN
-F 2 "MB_LIB:via" H 8450 1950 50  0001 C CNN
+F 2 "MB_LIB:via_sq" H 8450 1950 50  0001 C CNN
 F 3 "" H 8450 1950 50  0001 C CNN
 	1    8450 1950
@@
 $EndComp
 $Comp
-L Conn_01x03 J?
+L Conn_01x03 J17
 U 1 1 5AB02C89
 P 1700 6000
-F 0 "J?" H 1700 6200 50  0000 C CNN
+F 0 "J17" H 1700 6200 50  0000 C CNN
 F 1 "Conn_01x03" H 1700 5800 50  0000 C CNN
 F 2 "Connector_Molex:Molex_Panelmate_53780-0370_1x03_P1.25mm_Horizontal" H 1700 6000 50  0001 C CNN
@@
 NoConn ~ 1900 5900
 $Comp
-L GND #PWR?
+L GND #PWR033
 U 1 1 5AB02E47
 P 2000 6150
-F 0 "#PWR?" H 2000 5900 50  0001 C CNN
+F 0 "#PWR033" H 2000 5900 50  0001 C CNN
 F 1 "GND" H 2000 6000 50  0000 C CNN
 F 2 "" H 2000 6150 50  0001 C CNN
@@
 $EndComp
 $Comp
-L +12P #PWR?
+L +12P #PWR034
 U 1 1 5AB03206
 P 2000 5850
-F 0 "#PWR?" H 2000 5700 50  0001 C CNN
+F 0 "#PWR034" H 2000 5700 50  0001 C CNN
 F 1 "+12P" H 2000 5990 50  0000 C CNN
 F 2 "" H 2000 5850 50  0001 C CNN
@@
 	2000 6100 2000 6150
 $Comp
-L Conn_01x03 J?
+L Conn_01x03 J18
 U 1 1 5AB03435
 P 2300 6000
-F 0 "J?" H 2300 6200 50  0000 C CNN
+F 0 "J18" H 2300 6200 50  0000 C CNN
 F 1 "Conn_01x03" H 2300 5800 50  0000 C CNN
 F 2 "Connector_Molex:Molex_Panelmate_53780-0370_1x03_P1.25mm_Horizontal" H 2300 6000 50  0001 C CNN
@@
 NoConn ~ 2500 5900
 $Comp
-L GND #PWR?
+L GND #PWR035
 U 1 1 5AB0343C
 P 2600 6150
-F 0 "#PWR?" H 2600 5900 50  0001 C CNN
+F 0 "#PWR035" H 2600 5900 50  0001 C CNN
 F 1 "GND" H 2600 6000 50  0000 C CNN
 F 2 "" H 2600 6150 50  0001 C CNN
@@
 $EndComp
 $Comp
-L +12P #PWR?
+L +12P #PWR036
 U 1 1 5AB03442
 P 2600 5850
-F 0 "#PWR?" H 2600 5700 50  0001 C CNN
+F 0 "#PWR036" H 2600 5700 50  0001 C CNN
 F 1 "+12P" H 2600 5990 50  0000 C CNN
 F 2 "" H 2600 5850 50  0001 C CNN
@@
 	2600 6100 2600 6150
 $Comp
-L Conn_01x03 J?
+L Conn_01x03 J19
 U 1 1 5AB034A0
 P 2900 6000
-F 0 "J?" H 2900 6200 50  0000 C CNN
+F 0 "J19" H 2900 6200 50  0000 C CNN
 F 1 "Conn_01x03" H 2900 5800 50  0000 C CNN
 F 2 "Connector_Molex:Molex_Panelmate_53780-0370_1x03_P1.25mm_Horizontal" H 2900 6000 50  0001 C CNN
@@
 NoConn ~ 3100 5900
 $Comp
-L GND #PWR?
+L GND #PWR037
 U 1 1 5AB034A7
 P 3200 6150
-F 0 "#PWR?" H 3200 5900 50  0001 C CNN
+F 0 "#PWR037" H 3200 5900 50  0001 C CNN
 F 1 "GND" H 3200 6000 50  0000 C CNN
 F 2 "" H 3200 6150 50  0001 C CNN
@@
 $EndComp
 $Comp
-L +12P #PWR?
+L +12P #PWR038
 U 1 1 5AB034AD
 P 3200 5850
-F 0 "#PWR?" H 3200 5700 50  0001 C CNN
+F 0 "#PWR038" H 3200 5700 50  0001 C CNN
 F 1 "+12P" H 3200 5990 50  0000 C CNN
 F 2 "" H 3200 5850 50  0001 C CNN
@@
 	3200 6100 3200 6150
 $Comp
-L Conn_01x02 J?
+L Conn_01x02 J20
 U 1 1 5AB13823
 P 4300 5900
-F 0 "J?" H 4300 6000 50  0000 C CNN
+F 0 "J20" H 4300 6000 50  0000 C CNN
 F 1 "Conn_01x02" H 4300 5700 50  0000 C CNN
 F 2 "Connector_JST:JST_EH_S02B-EH_1x02_P2.50mm_Horizontal" H 4300 5900 50  0001 C CNN
@@
 $EndComp
 $Comp
-L GND #PWR?
+L GND #PWR039
 U 1 1 5AB13AC1
 P 4600 6100
-F 0 "#PWR?" H 4600 5850 50  0001 C CNN
+F 0 "#PWR039" H 4600 5850 50  0001 C CNN
 F 1 "GND" H 4600 5950 50  0000 C CNN
 F 2 "" H 4600 6100 50  0001 C CNN
@@
 $EndComp
 $Comp
-L GND #PWR?
+L GND #PWR040
 U 1 1 5AB13B2C
 P 5200 6100
-F 0 "#PWR?" H 5200 5850 50  0001 C CNN
+F 0 "#PWR040" H 5200 5850 50  0001 C CNN
 F 1 "GND" H 5200 5950 50  0000 C CNN
 F 2 "" H 5200 6100 50  0001 C CNN
@@
 $EndComp
 $Comp
-L GND #PWR?
+L GND #PWR041
 U 1 1 5AB13B97
 P 5800 6100
-F 0 "#PWR?" H 5800 5850 50  0001 C CNN
+F 0 "#PWR041" H 5800 5850 50  0001 C CNN
 F 1 "GND" H 5800 5950 50  0000 C CNN
 F 2 "" H 5800 6100 50  0001 C CNN
@@
 $EndComp
 $Comp
-L +5V #PWR?
+L +5V #PWR042
 U 1 1 5AB13D62
 P 4600 5800
-F 0 "#PWR?" H 4600 5650 50  0001 C CNN
+F 0 "#PWR042" H 4600 5650 50  0001 C CNN
 F 1 "+5V" H 4600 5940 50  0000 C CNN
 F 2 "" H 4600 5800 50  0001 C CNN
@@
 $EndComp
 $Comp
-L +5V #PWR?
+L +5V #PWR043
 U 1 1 5AB13EED
 P 5200 5800
-F 0 "#PWR?" H 5200 5650 50  0001 C CNN
+F 0 "#PWR043" H 5200 5650 50  0001 C CNN
 F 1 "+5V" H 5200 5940 50  0000 C CNN
 F 2 "" H 5200 5800 50  0001 C CNN
@@
 $EndComp
 $Comp
-L +5V #PWR?
+L +5V #PWR044
 U 1 1 5AB13F58
 P 5800 5800
-F 0 "#PWR?" H 5800 5650 50  0001 C CNN
+F 0 "#PWR044" H 5800 5650 50  0001 C CNN
 F 1 "+5V" H 5800 5940 50  0000 C CNN
 F 2 "" H 5800 5800 50  0001 C CNN
@@
 	5800 6000 5800 6100
 $Comp
-L Conn_01x02 J?
+L Conn_01x02 J21
 U 1 1 5AB14B61
 P 4900 5900
-F 0 "J?" H 4900 6000 50  0000 C CNN
+F 0 "J21" H 4900 6000 50  0000 C CNN
 F 1 "Conn_01x02" H 4900 5700 50  0000 C CNN
 F 2 "Connector_JST:JST_EH_S02B-EH_1x02_P2.50mm_Horizontal" H 4900 5900 50  0001 C CNN
@@
 $EndComp
 $Comp
-L Conn_01x02 J?
+L Conn_01x02 J22
 U 1 1 5AB14BDA
 P 5500 5900
-F 0 "J?" H 5500 6000 50  0000 C CNN
+F 0 "J22" H 5500 6000 50  0000 C CNN
 F 1 "Conn_01x02" H 5500 5700 50  0000 C CNN
 F 2 "Connector_JST:JST_EH_S02B-EH_1x02_P2.50mm_Horizontal" H 5500 5900 50  0001 C CNN

Commit message: new pcb design
Parts:
- added J23, J25: Conn_01x01, MB_LIB:via_sq, symbol Conn_01x01
- added J24, J26: Conn_01x01, MB_LIB:via, symbol Conn_01x01
Connections:
- net +12V: now also J25.1 (Pin_1)
- net +48V: now also J23.1 (Pin_1)
- net GND: now also J24.1 (Pin_1), J26.1 (Pin_1)
Changed lines of the file:
@@
 $EndComp
-Wire Wire Line
-	6100 2300 8450 2300
 Wire Wire Line
 	8450 2300 8450 2150
 Wire Wire Line
-	8150 2150 8150 2300
+	8150 2300 8150 2150
 Connection ~ 8150 2300
 Wire Wire Line
-	7850 2150 7850 2300
+	7850 2300 7850 2150
 Connection ~ 7850 2300
 Wire Wire Line
-	7550 2150 7550 2300
+	7550 2300 7550 2150
 Connection ~ 7550 2300
 Wire Wire Line
-	7250 2150 7250 2300
+	7250 2300 7250 2150
 Connection ~ 7250 2300
 Wire Wire Line
-	6950 2150 6950 2300
+	6950 2300 6950 2150
 Connection ~ 6950 2300
 Wire Wire Line
-	6650 2150 6650 2300
+	6650 2300 6650 2150
 Connection ~ 6650 2300
 Wire Wire Line
@@
 Wire Wire Line
 	6100 2700 6100 2550
-Wire Wire Line
-	6100 2550 8450 2550
 Wire Wire Line
 	8450 2550 8450 2700
@@
 	-1   0    0    -1
 $EndComp
+$Comp
+L Conn_01x01 J25
+U 1 1 5AC4894E
+P 7000 5850
+F 0 "J25" H 7000 5950 50  0000 C CNN
+F 1 "Conn_01x01" H 7000 5750 50  0000 C CNN
+F 2 "MB_LIB:via_sq" H 7000 5850 50  0001 C CNN
+F 3 "" H 7000 5850 50  0001 C CNN
+	1    7000 5850
+	-1   0    0    1
+$EndComp
+$Comp
+L Conn_01x01 J26
+U 1 1 5AC48954
+P 7000 6100
+F 0 "J26" H 7000 6200 50  0000 C CNN
+F 1 "Conn_01x01" H 7000 6000 50  0000 C CNN
+F 2 "MB_LIB:via" H 7000 6100 50  0001 C CNN
+F 3 "" H 7000 6100 50  0001 C CNN
+	1    7000 6100
+	-1   0    0    1
+$EndComp
+$Comp
+L Conn_01x01 J23
+U 1 1 5AC48C6B
+P 6450 5850
+F 0 "J23" H 6450 5950 50  0000 C CNN
+F 1 "Conn_01x01" H 6450 5750 50  0000 C CNN
+F 2 "MB_LIB:via_sq" H 6450 5850 50  0001 C CNN
+F 3 "" H 6450 5850 50  0001 C CNN
+	1    6450 5850
+	-1   0    0    1
+$EndComp
+$Comp
+L Conn_01x01 J24
+U 1 1 5AC48C71
+P 6450 6100
+F 0 "J24" H 6450 6200 50  0000 C CNN
+F 1 "Conn_01x01" H 6450 6000 50  0000 C CNN
+F 2 "MB_LIB:via" H 6450 6100 50  0001 C CNN
+F 3 "" H 6450 6100 50  0001 C CNN
+	1    6450 6100
+	-1   0    0    1
+$EndComp
+Wire Wire Line
+	6650 6100 6700 6100
+Wire Wire Line
+	6700 6100 6700 6150
+Wire Wire Line
+	6650 5850 6700 5850
+Wire Wire Line
+	6700 5850 6700 5700
+$Comp
+L +48V #PWR045
+U 1 1 5AC49110
+P 6700 5700
+F 0 "#PWR045" H 6700 5550 50  0001 C CNN
+F 1 "+48V" H 6700 5840 50  0000 C CNN
+F 2 "" H 6700 5700 50  0001 C CNN
+F 3 "" H 6700 5700 50  0001 C CNN
+	1    6700 5700
+	1    0    0    -1
+$EndComp
+$Comp
+L GND #PWR046
+U 1 1 5AC4916C
+P 6700 6150
+F 0 "#PWR046" H 6700 5900 50  0001 C CNN
+F 1 "GND" H 6700 6000 50  0000 C CNN
+F 2 "" H 6700 6150 50  0001 C CNN
+F 3 "" H 6700 6150 50  0001 C CNN
+	1    6700 6150
+	1    0    0    -1
+$EndComp
+Wire Wire Line
+	6100 2300 8450 2300
+Wire Wire Line
+	6100 2550 8450 2550
+Wire Wire Line
+	7250 5850 7200 5850
+Wire Wire Line
+	7250 5650 7250 5850
+$Comp
+L +12V #PWR047
+U 1 1 5AC4A9F4
+P 7250 5650
+F 0 "#PWR047" H 7250 5500 50  0001 C CNN
+F 1 "+12V" H 7250 5790 50  0000 C CNN
+F 2 "" H 7250 5650 50  0001 C CNN
+F 3 "" H 7250 5650 50  0001 C CNN
+	1    7250 5650
+	1    0    0    -1
+$EndComp
+Wire Wire Line
+	7200 6100 7250 6100
+Wire Wire Line
+	7250 6100 7250 6150
+$Comp
+L GND #PWR048
+U 1 1 5AC4AB14
+P 7250 6150
+F 0 "#PWR048" H 7250 5900 50  0001 C CNN
+F 1 "GND" H 7250 6000 50  0000 C CNN
+F 2 "" H 7250 6150 50  0001 C CNN
+F 3 "" H 7250 6150 50  0001 C CNN
+	1    7250 6150
+	1    0    0    -1
+$EndComp
 $EndSCHEMATC
