File: power_board.kicad_pcb (KiCad board)
At the start: 2 copper layers, 87.2 x 64 mm, 66 parts, among them J1 Conn_01x01, J10 Conn_01x01, J11 Conn_01x01, J12 Conn_01x01, J13 Conn_01x01, J14 Conn_01x01, J15 Conn_01x01, J16 Conn_01x01, J17 Conn_01x03, J18 Conn_01x03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

Commit message: new pcb design
Parts:
- removed the J16 at (54.4, 26.6)
- removed the J9 at (65.3, 26.3)
- added J23: Conn_01x01, MB_LIB:via_sq, F.Cu at (144.5, 103.2)
- added J24: Conn_01x01, MB_LIB:via, F.Cu at (144.6, 97.1)
- added J25: Conn_01x01, MB_LIB:via_sq, F.Cu at (134.2, 61.9)
- added J26: Conn_01x01, MB_LIB:via, F.Cu at (154.5, 61.7)
- Q2, Q3: moved to B.Cu
- moved Q2 121.8 mm to (169.0, 95.4)
- moved Q1 112.2 mm to (170.1, 51.8), turned to 90 degrees
- moved J10 98.1 mm to (166.0, 73.1), turned to 0 degrees
- moved J2 95.5 mm to (171.8, 67.3)
- moved J12 93.1 mm to (171.6, 73.1)
- moved J16 93.0 mm to (154.6, 73.1), turned to 0 degrees
- moved C2 84.5 mm to (157.4, 47.4), turned to 270 degrees
- moved Q3 74.9 mm to (120.2, 96.8), turned to 180 degrees
- moved J8 74.8 mm to (160.4, 73.1), turned to 0 degrees
- moved C7 71.2 mm to (144.1, 52.5), turned to 90 degrees
- moved J6 71.1 mm to (154.6, 67.4), turned to 0 degrees
- moved C4 69.1 mm to (170.2, 85.0), turned to 90 degrees
- moved J14 67.0 mm to (166.1, 67.4)
- moved J4 66.9 mm to (160.4, 67.4)
- moved D2 66.6 mm to (131.7, 96.3), turned to 180 degrees
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Other:
- board size 87.2 x 64 mm -> 68 x 76.7 mm

Commit message: routed
Parts:
- removed C1: 2m2, Capacitor_THT:CP_Radial_D12.5mm_P5.00mm
- added  : , MB_LIB:via, F.Cu at (139.8, 94.5)
- added  : , MB_LIB:via, F.Cu at (158.8, 110.9)
- added  : , MB_LIB:via, F.Cu at (158.0, 107.8)
- added  : , MB_LIB:via, F.Cu at (156.1, 107.7)
- added  : , MB_LIB:via, F.Cu at (135.3, 99.8)
- added  : , MB_LIB:via, F.Cu at (139.8, 99.9)
- added  : , MB_LIB:via, F.Cu at (127.8, 104.0)
- added  : , MB_LIB:via, F.Cu at (115.7, 103.7)
- added  : , MB_LIB:via, F.Cu at (115.4, 106.4)
- added  : , MB_LIB:via, F.Cu at (119.5, 109.4)
- added  : , MB_LIB:via, F.Cu at (121.5, 109.4)
- added  : , MB_LIB:via, F.Cu at (135.3, 94.5)
- added  : , MB_LIB:via, F.Cu at (112.8, 46.5)
- added  : , MB_LIB:via, F.Cu at (113.4, 48.4)
- added  : , MB_LIB:via, F.Cu at (126.4, 109.0)
- added  : , MB_LIB:via, F.Cu at (165.8, 107.1)
- added  : , MB_LIB:via, F.Cu at (125.8, 105.7)
- added  : , MB_LIB:via, F.Cu at (123.7, 107.2)
- added  : , MB_LIB:via, F.Cu at (122.2, 107.2)
- added  : , MB_LIB:via, F.Cu at (123.8, 104.2)
- added  : , MB_LIB:via, F.Cu at (122.3, 104.1)
- added  : , MB_LIB:via, F.Cu at (165.2, 105.5)
- added  : , MB_LIB:via, F.Cu at (173.4, 55.3)
- added  : , MB_LIB:via, F.Cu at (163.6, 105.5)
- added  : , MB_LIB:via, F.Cu at (163.4, 108.7)
- added  : , MB_LIB:via, F.Cu at (165.4, 108.6)
- added  : , MB_LIB:via, F.Cu at (167.8, 107.8)
- added  : , MB_LIB:via, F.Cu at (169.3, 106.2)
- added  : , MB_LIB:via, F.Cu at (169.6, 103.8)
- added  : , MB_LIB:via, F.Cu at (173.9, 103.3)
- added  : , MB_LIB:via, F.Cu at (173.6, 59.3)
- added  : , MB_LIB:via, F.Cu at (147.1, 112.9)
- added  : , MB_LIB:via, F.Cu at (158.2, 113.0)
- added  : , MB_LIB:via, F.Cu at (169.1, 113.0)
- added  : , MB_LIB:via, F.Cu at (169.8, 111.6)
- added  : , MB_LIB:via, F.Cu at (147.9, 111.5)
- moved R8 7.48 mm to (124.9, 108.7), turned to 90 degrees
- moved R9 5.94 mm to (125.9, 108.7), turned to 270 degrees
- moved C2 5.09 mm to (157.3, 52.5), turned to 90 degrees
- moved C22 4.60 mm to (129.1, 108.1), turned to 0 degrees
- moved C18 1.96 mm to (128.7, 104.4)
- moved C19 1.96 mm to (129.1, 106.7)
- moved R6 1.96 mm to (128.5, 105.4)
- moved C17 1.71 mm to (117.4, 105.1)
- moved C20 1.71 mm to (118.9, 108.1)
- moved C21 1.71 mm to (124.5, 103.0)
- moved R7 1.71 mm to (121.1, 108.7)
- moved U2 1.71 mm to (123.0, 105.7)
- moved R3 1.17 mm to (169.4, 108.2)
- moved C16 1.17 mm to (173.0, 106.5), turned to 90 degrees
- moved C12 1.17 mm to (169.9, 104.8)
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Routing:
- net /Overvoltage protection/GATE: track 0.00 -> 176.5 mm, vias 0 -> 7
- net +12P: track 0.00 -> 66.9 mm, vias 0 -> 2
- net +12V: track 0.00 -> 58.4 mm, vias 0 -> 6
- net +5V: track 0.00 -> 56.4 mm, vias 0 -> 2
- net +48V: track 0.00 -> 50.2 mm, vias 0 -> 2
- net Net-(C15-Pad1): track 0.00 -> 32.6 mm
- net GND: track 0.00 -> 27.8 mm, vias 0 -> 5
- net Net-(C21-Pad1): track 0.00 -> 13.3 mm
- net Net-(C19-Pad1): track 0.00 -> 4.63 mm
- net Net-(C13-Pad1): track 0.00 -> 4.04 mm
- net Net-(R3-Pad2): track 0.00 -> 3.72 mm
- net Net-(C21-Pad2): track 0.00 -> 3.39 mm
- net Net-(C20-Pad1): track 0.00 -> 2.60 mm
- net Net-(R8-Pad2): track 0.00 -> 2.06 mm
- net Net-(C14-Pad1): track 0.00 -> 1.54 mm
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- added copper zone on F.Cu, net +12V
- added copper zone on B.Cu, net GND
- added copper zone on F.Cu, net GND
- added copper zone on In1.Cu, net GND
- added copper zone on In2.Cu, net GND
Other:
- copper layers 2 -> 4
- rule trace_min: 0.2 -> 0.12

Commit message: PCB check
Parts:
- removed the   at (173.9, 103.3)
- moved C16 20.4 mm to (152.6, 106.2), turned to 270 degrees
- moved   0.61 mm to (164.9, 106.0)
- moved   0.59 mm to (165.2, 107.1)
- moved   0.56 mm to (163.8, 106.0)
- moved   0.50 mm to (164.9, 108.4)
- moved   0.48 mm to (163.8, 108.4)
Routing:
- net /Overvoltage protection/GATE: track 176.5 -> 10.4 mm, vias 7 -> 0
- net +12P: track 66.9 -> 6.17 mm, vias 2 -> 0
- net +12V: track 58.4 -> 6.00 mm, vias 6 -> 0
- net +5V: track 56.4 -> 4.87 mm, vias 2 -> 0
- net +48V: track 50.2 -> 32.3 mm, vias 2 -> 1
- net GND: track 27.8 -> 29.1 mm, vias 5 -> 4
Other:
- rule trace_min: 0.12 -> 0.16

Commit message: fixed
Parts:
- removed the   at (139.8, 94.5)
- removed the   at (158.8, 110.9)
- removed the   at (158.0, 107.8)
- removed the   at (156.1, 107.7)
- removed the   at (135.3, 99.8)
- removed the   at (139.8, 99.9)
- removed the   at (127.8, 104.0)
- removed the   at (115.7, 103.7)
- removed the   at (115.4, 106.4)
- removed the   at (119.5, 109.4)
- removed the   at (121.5, 109.4)
- removed the   at (135.3, 94.5)
- removed the   at (112.8, 46.5)
- removed the   at (113.4, 48.4)
- removed the   at (126.4, 109.0)
- removed the   at (165.2, 107.1)
- removed the   at (125.8, 105.7)
- removed the   at (123.7, 107.2)
- removed the   at (122.2, 107.2)
- removed the   at (123.8, 104.2)
- removed the   at (122.3, 104.1)
- removed the   at (164.9, 106.0)
- removed the   at (173.4, 55.3)
- removed the   at (163.8, 106.0)
- removed the   at (163.8, 108.4)
- removed the   at (164.9, 108.4)
- removed the   at (167.8, 107.8)
- removed the   at (169.3, 106.2)
- removed the   at (169.6, 103.8)
- removed the   at (173.6, 59.3)
- removed the   at (147.1, 112.9)
- removed the   at (158.2, 113.0)
- removed the   at (169.1, 113.0)
- removed the   at (169.8, 111.6)
- removed the   at (147.9, 111.5)
- added  : , MB_LIB:via, F.Cu at (108.6, 116.2)
- added  : , MB_LIB:via, F.Cu at (153.4, 109.2)
- added  : , MB_LIB:via, F.Cu at (153.5, 107.0)
- added  : , MB_LIB:via, F.Cu at (147.6, 111.9)
- added  : , MB_LIB:via, F.Cu at (147.5, 110.7)
- added  : , MB_LIB:via, F.Cu at (123.5, 106.4)
- added  : , MB_LIB:via, F.Cu at (122.3, 106.4)
- added  : , MB_LIB:via, F.Cu at (123.4, 104.8)
- added  : , MB_LIB:via, F.Cu at (122.2, 104.8)
- added  : , MB_LIB:via, F.Cu at (165.0, 107.9)
- added  : , MB_LIB:via, F.Cu at (163.7, 107.9)
- added  : , MB_LIB:via, F.Cu at (108.9, 46.8)
- added  : , MB_LIB:via, F.Cu at (165.1, 106.1)
- added  : , MB_LIB:via, F.Cu at (163.6, 106.1)
- added  : , MB_LIB:via, F.Cu at (159.1, 107.1)
- added  : , MB_LIB:via, F.Cu at (160.1, 109.2)
- added  : , MB_LIB:via, F.Cu at (167.7, 107.7)
- added  : , MB_LIB:via, F.Cu at (170.5, 106.3)
- added  : , MB_LIB:via, F.Cu at (170.3, 103.9)
- added  : , MB_LIB:via, F.Cu at (139.6, 98.2)
- added  : , MB_LIB:via, F.Cu at (135.3, 98.2)
- added  : , MB_LIB:via, F.Cu at (135.4, 94.5)
- added  : , MB_LIB:via, F.Cu at (176.8, 111.2)
- added  : , MB_LIB:via, F.Cu at (139.7, 94.5)
- added  : , MB_LIB:via, F.Cu at (116.6, 103.8)
- added  : , MB_LIB:via, F.Cu at (116.6, 106.4)
- added  : , MB_LIB:via, F.Cu at (121.4, 109.4)
- added  : , MB_LIB:via, F.Cu at (119.5, 109.3)
- added  : , MB_LIB:via, F.Cu at (126.5, 108.9)
- added  : , MB_LIB:via, F.Cu at (126.0, 105.7)
- added  : , MB_LIB:via, F.Cu at (127.5, 104.4)
- added  : , MB_LIB:via, F.Cu at (130.4, 106.3)
- added  : , MB_LIB:via, F.Cu at (132.5, 109.8)
- added  : , MB_LIB:via, F.Cu at (176.6, 62.7)
- added  : , MB_LIB:via, F.Cu at (132.4, 107.8)
- added  : , MB_LIB:via, F.Cu at (158.8, 112.2)
- added  : , MB_LIB:via, F.Cu at (158.6, 110.7)
- added  : , MB_LIB:via, F.Cu at (169.4, 112.3)
- added  : , MB_LIB:via, F.Cu at (169.4, 110.8)
- added  : , MB_LIB:via, F.Cu at (176.2, 89.3)
- added  : , MB_LIB:via, F.Cu at (173.4, 59.4)
- added  : , MB_LIB:via, F.Cu at (173.5, 55.2)
- added  : , MB_LIB:via, F.Cu at (112.8, 46.5)
- added  : , MB_LIB:via, F.Cu at (114.5, 52.7)
- added  : , MB_LIB:via, F.Cu at (114.8, 48.7)
- C22: footprint Capacitors_SMD:C_0603 -> Capacitor_SMD:C_1206_3216Metric_Pad1.24x1.80mm_HandSolder
- moved C22 1.18 mm to (130.0, 108.9)
Routing:
- net /Overvoltage protection/GATE: track 10.4 -> 155.6 mm, vias 0 -> 5
- net +12V: track 6.00 -> 85.4 mm
- net +12P: track 6.17 -> 70.7 mm
- net +5V: track 4.87 -> 58.1 mm
- net +48V: track 32.3 -> 49.8 mm, vias 1 -> 2
- added copper zone on B.Cu, net +12V
- added copper zone on In1.Cu, net +12V
- added copper zone on In2.Cu, net +12V
Other:
- board size 68 x 76.7 mm -> 73.6 x 76.8 mm

Commit message: now its good ?
Parts:
- moved   3.97 mm to (179.7, 60.1)
- moved   3.28 mm to (179.0, 113.6)
- moved   1.03 mm to (107.6, 116.0)
- moved   0.96 mm to (108.0, 47.2)
Routing:
- net /Overvoltage protection/GATE: track 155.6 -> 166.7 mm
Other:
- board size 73.6 x 76.8 mm -> 80 x 76.7 mm
